Commit message: Remove collision from caster hub
  - Update joint axis
  - Update wheel friction

File: htb_description/urdf/caster.xacro (robot description, xacro)
@@ -9,5 +9,5 @@
       <joint_properties damping="0.0" friction="0.0" />
       <parent link="link_chassis"/>
-        <axis rpy="0 0 0" xyz="0 1 0"/>
+        <axis rpy="0 0 0" xyz="0 0 1"/>
       <child link="caster_${wheel}_swivel"/>
     </joint>
@@ -49,10 +49,4 @@
         </material>
       </visual>
-      <collision>
-        <origin xyz="0 0 0" rpy="0 0 0"/>
-        <geometry>
-          <box size="0.05 0.05 0.05"/>
-        </geometry>
-      </collision>
     </link>
     <gazebo reference="caster_hubcap">
@@ -85,9 +79,20 @@
       </visual>
       <collision>
-        <origin xyz="0 0 0" rpy="${-3.1415927/2.0} 0 0"/>
+        <!-- <origin xyz="0 0 0" rpy="${-3.1415927/2.0} 0 0"/> -->
+        <origin xyz="0 0 0" rpy="0 0 0"/>
         <geometry>
           <mesh filename="package://htb_description/meshes/caster_wheel.stl"/>
           <cylinder radius="0.0375" length="0.01"/>
         </geometry>
+        <surface>
+          <friction>
+            <ode>
+              <mu>0.01</mu>
+              <mu2>0.1</mu2>
+              <slip1>1.0</slip1>
+              <slip2>1.0</slip2>
+            </ode>
+          </friction>
+        </surface>
       </collision>
     </link>

File: htb_description/urdf/htb.xacro (robot description, xacro)
@@ -100,5 +100,5 @@
   <xacro:link_wheel name="link_left_wheel" />
   <xacro:joint_wheel name="joint_left_wheel" child="link_left_wheel" origin_xyz="-0.125 0.2225 -0.04" />
-  <xacro:caster_wheel name="left_caster" origin_xyz="0.185 0.11 -0.08" wheel="l"/>
-  <xacro:caster_wheel name="right_caster" origin_xyz="0.185 -0.11 -0.08" wheel="r"/>
+  <xacro:caster_wheel name="left_caster" origin_xyz="0.185 0.11 -0.06" wheel="l"/>
+  <xacro:caster_wheel name="right_caster" origin_xyz="0.185 -0.11 -0.06" wheel="r"/>
 </robot>

Commit message: Update swivel colors

File: htb_description/urdf/caster.xacro (robot description, xacro)
@@ -24,12 +24,7 @@
           <mesh filename="package://htb_description/meshes/caster_swivel.stl"/>
         </geometry>
-        <material name="caster_${wheel}_swivel">
-          <color rgba="0.5 0.5 0.5 1"/>
-        </material>
+        <material name="blue"/>
       </visual>
     </link>
-    <gazebo reference="caster_swivel">
-      <material value="Gazebo/Grey"/>
-    </gazebo>
     <!-- Center Wheel + Hubcap -->
     <link name="caster_${wheel}_hubcap">
@@ -45,12 +40,7 @@
           <mesh filename="package://htb_description/meshes/caster_hubcap.stl"/>
         </geometry>
-        <material name="caster_${wheel}_swivel">
-          <color rgba="0.5 0.5 0.5 1"/>
-        </material>
+        <material name="blue"/>
       </visual>
     </link>
-    <gazebo reference="caster_hubcap">
-      <material value="Gazebo/Grey"/>
-    </gazebo>
     <joint name="caster_${wheel}_swivel_hubcap_joint" type="continuous">
       <origin xyz="-0.026 0 -0.016" rpy="0 0 0"/>

Commit message: Move from link_chassis to base_link

File: htb_description/urdf/caster.xacro (robot description, xacro)
@@ -8,5 +8,5 @@
       <limit effort="100" velocity="100" k_velocity="0" />
       <joint_properties damping="0.0" friction="0.0" />
-      <parent link="link_chassis"/>
+      <parent link="base_link"/>
         <axis rpy="0 0 0" xyz="0 0 1"/>
       <child link="caster_${wheel}_swivel"/>

File: htb_description/urdf/htb.xacro (robot description, xacro)
@@ -6,5 +6,5 @@
   <xacro:include filename="$(find htb_description)/urdf/caster.xacro" />
   <xacro:property name="camera_link_size" value="0.05" /> <!-- Size of square 'camera' box -->
-  <link name="link_chassis">
+  <link name="base_link">
     <!-- pose and inertial -->
     <pose>0 0 0.11 0 0 0</pose>
@@ -32,5 +32,5 @@
     <axis xyz="0 1 0" />
     <origin xyz="-0.21 0 0.01" rpy="0 0 0"/>
-    <parent link="link_chassis"/>
+    <parent link="base_link"/>
     <child link="v_support_link"/>
   </joint>
@@ -60,5 +60,5 @@
     <axis xyz="0 1 0" />
     <origin xyz="0.215 0 0.01" rpy="0 0 0"/>
-    <parent link="link_chassis"/>
+    <parent link="base_link"/>
     <child link="rplidar_link"/>
   </joint>
@@ -88,5 +88,5 @@
     <axis xyz="0 1 0" />
     <origin xyz="-0.215 0 0.8" rpy="0 0 0"/>
-    <parent link="link_chassis"/>
+    <parent link="base_link"/>
     <child link="realsense_camera"/>
   </joint>

File: htb_description/urdf/macros.xacro (robot description, xacro)
@@ -27,5 +27,5 @@
         <origin rpy="0 0 0" xyz="${origin_xyz}"/>
         <child link="${child}"/>
-        <parent link="link_chassis"/>
+        <parent link="base_link"/>
         <axis rpy="0 0 0" xyz="0 1 0"/>
         <limit effort="10000" velocity="1000"/>
