Commit message: Update wheel distance and colors

File: htb_description/urdf/htb.xacro (robot description, xacro)
@@ -27,6 +27,6 @@
     </visual>
     <!-- caster front left-->
-    <collision name="caster_front_collision">
-      <origin rpy=" 0 0 0" xyz="0.35 0 -0.05"/>
+    <collision name="caster_front_left_collision">
+      <origin rpy=" 0 0 0" xyz="0.185 0.11 -0.05"/>
       <geometry>
         <sphere radius="0.05"/>
@@ -43,6 +43,29 @@
       </surface>
     </collision>
-    <visual name="caster_front_visual">
-      <origin rpy=" 0 0 0" xyz="0.2 0 -0.05"/>
+    <visual name="caster_front_left_visual">
+      <origin rpy=" 0 0 0" xyz="0.185 0.11 -0.05"/>
+      <geometry>
+        <sphere radius="0.05"/>
+      </geometry>
+    </visual>
+    <!-- caster front right-->
+    <collision name="caster_front_right_collision">
+      <origin rpy=" 0 0 0" xyz="0.185 -0.11 -0.05"/>
+      <geometry>
+        <sphere radius="0.05"/>
+      </geometry>
+      <surface>
+        <friction>
+          <ode>
+            <mu>0</mu>
+            <mu2>0</mu2>
+            <slip1>1.0</slip1>
+            <slip2>1.0</slip2>
+          </ode>
+        </friction>
+      </surface>
+    </collision>
+    <visual name="caster_front_right_visual">
+      <origin rpy=" 0 0 0" xyz="0.185 -0.11 -0.05"/>
       <geometry>
         <sphere radius="0.05"/>
@@ -70,5 +93,5 @@
         <box size="0.02 0.02 1.0"/>
       </geometry>
-      <material name="red"/>
+      <material name="grey"/>
     </visual>
     <inertial>

Commit message: Add caster wheel

File: htb_description/urdf/htb.xacro (robot description, xacro)
@@ -4,4 +4,5 @@
   <xacro:include filename="$(find htb_description)/urdf/htb.gazebo" />
   <xacro:include filename="$(find htb_description)/urdf/macros.xacro" />
+  <xacro:include filename="$(find htb_description)/urdf/caster.xacro" />
   <xacro:property name="camera_link_size" value="0.05" /> <!-- Size of square 'camera' box -->
   <link name="link_chassis">
@@ -25,50 +26,4 @@
       </geometry>
       <material name="blue"/>
-    </visual>
-    <!-- caster front left-->
-    <collision name="caster_front_left_collision">
-      <origin rpy=" 0 0 0" xyz="0.185 0.11 -0.05"/>
-      <geometry>
-        <sphere radius="0.05"/>
-      </geometry>
-      <surface>
-        <friction>
-          <ode>
-            <mu>0</mu>
-            <mu2>0</mu2>
-            <slip1>1.0</slip1>
-            <slip2>1.0</slip2>
-          </ode>
-        </friction>
-      </surface>
-    </collision>
-    <visual name="caster_front_left_visual">
-      <origin rpy=" 0 0 0" xyz="0.185 0.11 -0.05"/>
-      <geometry>
-        <sphere radius="0.05"/>
-      </geometry>
-    </visual>
-    <!-- caster front right-->
-    <collision name="caster_front_right_collision">
-      <origin rpy=" 0 0 0" xyz="0.185 -0.11 -0.05"/>
-      <geometry>
-        <sphere radius="0.05"/>
-      </geometry>
-      <surface>
-        <friction>
-          <ode>
-            <mu>0</mu>
-            <mu2>0</mu2>
-            <slip1>1.0</slip1>
-            <slip2>1.0</slip2>
-          </ode>
-        </friction>
-      </surface>
-    </collision>
-    <visual name="caster_front_right_visual">
-      <origin rpy=" 0 0 0" xyz="0.185 -0.11 -0.05"/>
-      <geometry>
-        <sphere radius="0.05"/>
-      </geometry>
     </visual>
   </link>
@@ -145,3 +100,5 @@
   <xacro:link_wheel name="link_left_wheel" />
   <xacro:joint_wheel name="joint_left_wheel" child="link_left_wheel" origin_xyz="-0.125 0.2225 -0.04" />
+  <xacro:caster_wheel name="left_caster" origin_xyz="0.185 0.11 -0.08" wheel="l"/>
+  <xacro:caster_wheel name="right_caster" origin_xyz="0.185 -0.11 -0.08" wheel="r"/>
 </robot>

File: htb_description/urdf/macros.xacro (robot description, xacro)
@@ -1,4 +1,5 @@
 <?xml version="1.0"?>
 <robot xmlns:xacro="http://www.ros.org/wiki/xacro">
+  <!-- Inspired by https://github.com/MobileRobots/amr-ros-config -->
     <xacro:macro name="link_wheel" params="name">
         <link name="${name}">

Commit message: Rotate realsense collision origin

File: htb_description/urdf/htb.xacro (robot description, xacro)
@@ -66,5 +66,5 @@
   <link name="camera_link">
     <collision>
-      <origin xyz="0 0 0" rpy="0 0 0"/>
+      <origin xyz="0.03 0 0" rpy="${-pi/2} 0 ${-pi/2}"/>
       <geometry>
         <mesh filename="package://htb_description/meshes/realsense.dae"/>

Commit message: Rename link to avoid overlap

File: htb_description/urdf/htb.xacro (robot description, xacro)
@@ -61,8 +61,8 @@
     <origin xyz="-0.21 0 0.8" rpy="0 0 0"/>
     <parent link="link_chassis"/>
-    <child link="camera_link"/>
+    <child link="realsense_camera"/>
   </joint>
   <!-- Camera link-->
-  <link name="camera_link">
+  <link name="realsense_camera">
     <collision>
       <origin xyz="0.03 0 0" rpy="${-pi/2} 0 ${-pi/2}"/>
@@ -90,8 +90,15 @@
         won't be aligned properly with the frame it is supposedly originating from -->
     <origin xyz="0 0 0" rpy="${-pi/2} 0 ${-pi/2}"/>
-    <parent link="camera_link"/>
-    <child link="camera_link_optical"/>
+    <parent link="realsense_camera"/>
+    <child link="realsense_link_optical"/>
   </joint>
-  <link name="camera_link_optical">
+  <link name="realsense_link_optical">
+  </link>
+  <joint name="realsense_mountpoint_joint" type="fixed">
+    <origin xyz="0 0 0" rpy="0 0 0"/>
+    <parent link="realsense_link_optical"/>
+    <child link="realsense_mount_point"/>
+  </joint>
+  <link name="realsense_mount_point">
   </link>
   <!-- -->

Commit message: Change camera link

File: htb_description/urdf/htb.xacro (robot description, xacro)
@@ -97,5 +97,5 @@
   <joint name="realsense_mountpoint_joint" type="fixed">
     <origin xyz="0 0 0" rpy="0 0 0"/>
-    <parent link="realsense_link_optical"/>
+    <parent link="realsense_camera"/>
     <child link="realsense_mount_point"/>
   </joint>

Commit message: Add rplidar link and 3D model

File: htb_description/urdf/htb.xacro (robot description, xacro)
@@ -56,8 +56,36 @@
     </inertial>
   </link>
+  <!-- RP-lidar joint-->
+  <joint name="rplidar_joint" type="fixed">
+    <axis xyz="0 1 0" />
+    <origin xyz="0.215 0 0.01" rpy="0 0 0"/>
+    <parent link="link_chassis"/>
+    <child link="rplidar_link"/>
+  </joint>
+  <!-- RP-lidar link-->
+  <link name="rplidar_link">
+    <collision>
+      <origin xyz="0 0 0" rpy="0 0 0"/>
+      <geometry>
+        <mesh filename="package://htb_description/meshes/rplidar.dae"/>
+      </geometry>
+    </collision>
+    <visual>
+      <origin xyz="0 0 0" rpy="0 0 0"/>
+      <geometry>
+        <mesh filename="package://htb_description/meshes/rplidar.dae"/>
+      </geometry>
+      <material name="red"/>
+    </visual>
+    <inertial>
+      <mass value="1e-5" />
+      <origin xyz="0 0 0" rpy="0 0 0"/>
+      <inertia ixx="1e-6" ixy="0" ixz="0" iyy="1e-6" iyz="0" izz="1e-6" />
+    </inertial>
+  </link>
   <!-- Camera joint-->
   <joint name="camera_joint" type="fixed">
     <axis xyz="0 1 0" />
-    <origin xyz="-0.21 0 0.8" rpy="0 0 0"/>
+    <origin xyz="-0.215 0 0.8" rpy="0 0 0"/>
     <parent link="link_chassis"/>
     <child link="realsense_camera"/>

Commit message: Update rplidar axis looking front

File: htb_description/urdf/htb.xacro (robot description, xacro)
@@ -59,5 +59,5 @@
   <joint name="rplidar_joint" type="fixed">
     <axis xyz="0 1 0" />
-    <origin xyz="0.215 0 0.01" rpy="0 0 0"/>
+    <origin xyz="0.215 0 0.01" rpy="0 0 ${pi}"/>
     <parent link="base_link"/>
     <child link="rplidar_link"/>

Commit message: Add rplidar sensor

File: htb_description/urdf/htb.xacro (robot description, xacro)
@@ -1,6 +1,6 @@
 <?xml version="1.0" ?>
 <robot name="htb" xmlns:xacro="http://www.ros.org/wiki/xacro">
+  <xacro:include filename="$(find htb_description)/urdf/htb.gazebo" />
   <xacro:include filename="$(find htb_description)/urdf/materials.xacro" />
-  <xacro:include filename="$(find htb_description)/urdf/htb.gazebo" />
   <xacro:include filename="$(find htb_description)/urdf/macros.xacro" />
   <xacro:include filename="$(find htb_description)/urdf/caster.xacro" />
@@ -59,5 +59,5 @@
   <joint name="rplidar_joint" type="fixed">
     <axis xyz="0 1 0" />
-    <origin xyz="0.215 0 0.01" rpy="0 0 ${pi}"/>
+    <origin xyz="0.215 0 0.06" rpy="0 0 ${pi}"/>
     <parent link="base_link"/>
     <child link="rplidar_link"/>
@@ -66,5 +66,5 @@
   <link name="rplidar_link">
     <collision>
-      <origin xyz="0 0 0" rpy="0 0 0"/>
+      <origin xyz="0 0 -0.06" rpy="0 0 ${pi}"/>
       <geometry>
         <mesh filename="package://htb_description/meshes/rplidar.dae"/>
@@ -72,5 +72,5 @@
     </collision>
     <visual>
-      <origin xyz="0 0 0" rpy="0 0 0"/>
+      <origin xyz="0 0 -0.06" rpy="0 0 ${pi}"/>
       <geometry>
         <mesh filename="package://htb_description/meshes/rplidar.dae"/>

Commit message: Update robot model

File: htb_description/urdf/htb.xacro (robot description, xacro)
@@ -28,36 +28,32 @@
     </visual>
   </link>
-  <!-- Vertical support joint-->
-  <joint name="v_support_joint" type="fixed">
+  <!-- upper joint-->
+  <joint name="upper_joint" type="fixed">
     <axis xyz="0 1 0" />
-    <origin xyz="-0.21 0 0.01" rpy="0 0 0"/>
+    <origin xyz="0 0 0.14" rpy="0 0 0"/>
     <parent link="base_link"/>
-    <child link="v_support_link"/>
+    <child link="upper_link"/>
   </joint>
-  <!-- v support link-->
-  <link name="v_support_link">
-    <collision>
-      <origin xyz="0 0 0.5" rpy="0 0 0"/>
+  <link name="upper_link">
+    <!-- pose and inertial -->
+    <pose>0 0 0.11 0 0 0</pose>
+    <inertial>
+      <mass value="2"/>
+      <origin rpy="0 0 0" xyz="0 0 0.11"/>
+      <inertia ixx="0.0395416666667" ixy="0" ixz="0" iyy="0.106208333333" iyz="0" izz="0.106208333333"/>
+    </inertial>
+    <!-- body -->
+    <visual>
+      <origin rpy="0 0 0" xyz="0 0 0"/>
       <geometry>
-        <box size="0.02 0.02 1.0"/>
+        <box size="0.53 0.38 0.02"/>
       </geometry>
-    </collision>
-    <visual>
-      <origin xyz="0 0 0.5" rpy="0 0 0"/>
-      <geometry>
-        <box size="0.02 0.02 1.0"/>
-      </geometry>
-      <material name="grey"/>
+      <material name="blue"/>
     </visual>
-    <inertial>
-      <mass value="1e-5" />
-      <origin xyz="0 0 0" rpy="0 0 0"/>
-      <inertia ixx="1e-6" ixy="0" ixz="0" iyy="1e-6" iyz="0" izz="1e-6" />
-    </inertial>
   </link>
   <!-- RP-lidar joint-->
   <joint name="rplidar_joint" type="fixed">
     <axis xyz="0 1 0" />
-    <origin xyz="0.215 0 0.06" rpy="0 0 ${pi}"/>
+    <origin xyz="0.215 0 0.12" rpy="0 0 ${pi}"/>
     <parent link="base_link"/>
     <child link="rplidar_link"/>
@@ -87,5 +83,5 @@
   <joint name="camera_joint" type="fixed">
     <axis xyz="0 1 0" />
-    <origin xyz="-0.215 0 0.8" rpy="0 0 0"/>
+    <origin xyz="0.145 0.125 0.10" rpy="0 0 0"/>
     <parent link="base_link"/>
     <child link="realsense_camera"/>
@@ -137,3 +133,7 @@
   <xacro:caster_wheel name="left_caster" origin_xyz="0.185 0.11 -0.06" wheel="l"/>
   <xacro:caster_wheel name="right_caster" origin_xyz="0.185 -0.11 -0.06" wheel="r"/>
+  <xacro:vertical_support number="1" x="0.105"  y="0.17" />
+  <xacro:vertical_support number="2" x="0.105"  y="-0.17" />
+  <xacro:vertical_support number="3" x="-0.245" y="0.17"  />
+  <xacro:vertical_support number="4" x="-0.245" y="-0.17"  />
 </robot>

File: htb_description/urdf/macros.xacro (robot description, xacro)
@@ -38,3 +38,30 @@
                 izz="${mass*(r*r)/2}" />
     </xacro:macro>
-</robot>
+    <xacro:macro name="vertical_support" params="number x y">
+      <link name="support_${number}">
+        <inertial>
+          <mass value="0.1"/>
+          <origin xyz="0 0 0" rpy="0 0 0"/>
+          <inertia ixx="0.000526666666667" ixy="0" ixz="0" iyy="0.000526666666667" iyz="0" izz="0.001"/>
+        </inertial>
+        <collision name="vertical_support_${number}_collision">
+          <origin xyz="0 0 0" rpy="0 0 0"/>
+          <geometry>
+            <box size="0.04 0.04 0.12"/>
+          </geometry>
+        </collision>
+        <visual name="support_${number}_visual">
+          <origin xyz="0 0 0" rpy="0 0 0"/>
+          <geometry>
+            <box size="0.04 0.04 0.12"/>
+          </geometry>
+        </visual>
+      </link>
+      <joint name="support_${number}_joint" type="fixed">
+        <axis xyz="0 0 1" />
+        <origin rpy="0 0 0" xyz="${x} ${y} 0.07"/>
+        <parent link="base_link"/>
+        <child link="support_${number}"/>
+      </joint>
+    </xacro:macro>
+  </robot>

Commit message: Fix rplidar orientation

File: htb_description/urdf/htb.xacro (robot description, xacro)
@@ -55,5 +55,5 @@
   <joint name="rplidar_joint" type="fixed">
     <axis xyz="0 1 0" />
-    <origin xyz="0.215 0 0.12" rpy="0 0 ${pi}"/>
+    <origin xyz="0.215 0 0.12" rpy="0 0 0"/>
     <parent link="base_link"/>
     <child link="rplidar_link"/>

Commit message: Update wheel position and realsense support

File: htb_description/urdf/htb.xacro (robot description, xacro)
@@ -83,6 +83,6 @@
   <joint name="camera_joint" type="fixed">
     <axis xyz="0 1 0" />
-    <origin xyz="-0.21 0 0.8" rpy="0 0 0"/>
-    <parent link="link_chassis"/>
+    <origin xyz="0.22 0.08 0.10" rpy="0 0 0"/>
+    <parent link="base_link"/>
     <child link="realsense_camera"/>
   </joint>
@@ -128,9 +128,9 @@
   <!-- -->
   <xacro:link_wheel name="link_right_wheel" />
-  <xacro:joint_wheel name="right_wheel" child="link_right_wheel" origin_xyz="-0.125 -0.2225 -0.04" />
+  <xacro:joint_wheel name="right_wheel" child="link_right_wheel" origin_xyz="0.125 -0.2225 -0.04" />
   <xacro:link_wheel name="link_left_wheel" />
-  <xacro:joint_wheel name="left_wheel" child="link_left_wheel" origin_xyz="-0.125 0.2225 -0.04" />
-  <xacro:caster_wheel name="left_caster" origin_xyz="0.185 0.11 -0.06" wheel="l"/>
-  <xacro:caster_wheel name="right_caster" origin_xyz="0.185 -0.11 -0.06" wheel="r"/>
+  <xacro:joint_wheel name="left_wheel" child="link_left_wheel" origin_xyz="0.125 0.2225 -0.04" />
+  <xacro:caster_wheel name="left_caster" origin_xyz="-0.185 0.11 -0.06" wheel="l"/>
+  <xacro:caster_wheel name="right_caster" origin_xyz="-0.185 -0.11 -0.06" wheel="r"/>
   <xacro:vertical_support number="1" x="0.105"  y="0.17" />
   <xacro:vertical_support number="2" x="0.105"  y="-0.17" />
