Commit message: Update robot description and plugins

File: htb_description/urdf/gazebo_control.xacro (robot description, xacro)
@@ -3,12 +3,15 @@
     <gazebo>
         <plugin name="diff_drive" filename="libgazebo_ros_diff_drive.so">
-            <!-- Wheel Information -->
+            <!-- Wheels -->
             <left_joint>left_wheel_joint</left_joint>
             <right_joint>right_wheel_joint</right_joint>
+            <!-- Kinematics -->
             <wheel_separation>0.45</wheel_separation>
             <wheel_diameter>0.16</wheel_diameter>
             <!-- Limits -->
-            <max_wheel_torque>200</max_wheel_torque>
-            <max_wheel_acceleration>10.0</max_wheel_acceleration>
+            <max_wheel_torque>20</max_wheel_torque>
+            <max_wheel_acceleration>1.0</max_wheel_acceleration>
+            <!-- Input -->
+            <!-- <commandTopic>cmd_velo</commandTopic> -->
             <!-- Output -->
             <odometry_frame>odom</odometry_frame>

File: htb_description/urdf/htb.urdf.xacro (robot description, xacro)
@@ -1,11 +1,10 @@
 <?xml version="1.0" ?>
 <robot name="htb" xmlns:xacro="http://www.ros.org/wiki/xacro">
-  <xacro:include filename="$(find htb_description)/urdf/ros2_control.xacro" />
   <xacro:include filename="$(find htb_description)/urdf/materials.urdf.xacro" />
   <xacro:include filename="$(find htb_description)/urdf/mech/wheel.urdf.xacro" />
   <xacro:include filename="$(find htb_description)/urdf/mech/caster.urdf.xacro" />
   <xacro:property name="camera_link_size" value="0.05" /> <!-- Size of square 'camera' box -->
-  <xacro:arg name="use_ros2_control" default="true"/>
-  <xacro:arg name="sim_mode" default="true"/>
+  <xacro:arg name="use_ros2_control" default="false" />
+  <xacro:arg name="sim_mode" default="true" />
   <link name="base_link">
     <!-- pose and inertial -->
@@ -39,5 +38,6 @@
   <link name="upper_link">
     <!-- pose and inertial -->
-    <pose>0 0 0.11 0 0 0</pose>
+    <pose>0
+      0 0.11 0 0 0</pose>
     <inertial>
       <mass value="2"/>
@@ -143,9 +143,9 @@
   <xacro:vertical_support number="3" x="-0.245" y="0.17"  />
   <xacro:vertical_support number="4" x="-0.245" y="-0.17"  />
-  <!-- <xacro:if value="$(arg use_ros2_control)">
-      <xacro:include filename="ros2_control.xacro" />
-  </xacro:if> -->
-  <!-- <xacro:unless value="$(arg use_ros2_control)">
-      <xacro:include filename="gazebo_control.xacro" />
-  </xacro:unless> -->
+  <xacro:if value="$(arg use_ros2_control)">
+    <xacro:include filename="$(find htb_description)/urdf/ros2_control.xacro" />
+  </xacro:if>
+  <xacro:unless value="$(arg use_ros2_control)">
+    <xacro:include filename="$(find htb_description)/urdf/gazebo_control.xacro" />
+  </xacro:unless>
 </robot>

File: htb_description/urdf/mech/caster.urdf.xacro (robot description, xacro)
@@ -21,5 +21,5 @@
       <visual>
         <origin xyz="0 0 0" rpy="0 0 0"/>
-        <geometry name="htb_geom">
+        <geometry name="base_link">
           <mesh filename="package://htb_description/meshes/caster_swivel.stl"/>
         </geometry>
@@ -37,5 +37,5 @@
       <visual>
         <origin xyz="0 0 0" rpy="0 0 0"/>
-        <geometry name="htb_geom">
+        <geometry name="base_link">
           <mesh filename="package://htb_description/meshes/caster_hubcap.stl"/>
         </geometry>
@@ -61,5 +61,5 @@
       <visual>
         <origin xyz="0 0 0" rpy="0 0 0"/>
-        <geometry name="htb_geom">
+        <geometry name="base_link">
           <mesh filename="package://htb_description/meshes/caster_wheel.stl"/>
         </geometry>

File: htb_description/urdf/mech/wheel.urdf.xacro (robot description, xacro)
@@ -28,6 +28,4 @@
         <parent link="base_link"/>
         <axis rpy="0 0 0" xyz="0 1 0"/>
-        <limit effort="10000" velocity="1000"/>
-        <joint_properties damping="1.0" friction="1.0"/>
       </joint>
     </xacro:macro>

File: htb_description/urdf/ros2_control.xacro (robot description, xacro)
@@ -1,8 +1,8 @@
 <?xml version="1.0"?>
 <robot xmlns:xacro="http://ros.org/wiki/xacro">
+  <!-- Real robot plugin -->
   <xacro:unless value="$(arg sim_mode)">
     <ros2_control name="GazeboSystem" type="system">
       <hardware>
-        <!-- Real robot plugin to modify -->
         <plugin>gazebo_ros2_control/GazeboSystem</plugin>
       </hardware>
@@ -25,4 +25,5 @@
     </ros2_control>
   </xacro:unless>
+  <!-- Simulated robot -->
   <xacro:if value="$(arg sim_mode)">
     <ros2_control name="GazeboSystem" type="system">
