Commit message: Add meshes dependencies

File: htb_description/urdf/htb.urdf.xacro (robot description, xacro)
@@ -64,5 +64,5 @@
       <origin xyz="0 0 -0.06" rpy="0 0 ${pi}"/>
       <geometry>
-        <mesh filename="package://htb_description/meshes/rplidar.dae"/>
+        <mesh filename="file://$(find htb_description)/meshes/rplidar.dae"/>
       </geometry>
     </collision>
@@ -70,5 +70,5 @@
       <origin xyz="0 0 -0.06" rpy="0 0 ${pi}"/>
       <geometry>
-        <mesh filename="package://htb_description/meshes/rplidar.dae"/>
+        <mesh filename="file://$(find htb_description)/meshes/rplidar.dae"/>
       </geometry>
       <material name="red"/>
@@ -92,5 +92,5 @@
       <origin xyz="0.03 0 0" rpy="${-pi/2} 0 ${-pi/2}"/>
       <geometry>
-        <mesh filename="package://htb_description/meshes/realsense.dae"/>
+        <mesh filename="file://$(find htb_description)/meshes/realsense.dae"/>
       </geometry>
     </collision>
@@ -98,5 +98,5 @@
       <origin xyz="0.03 0 0" rpy="${-pi/2} 0 ${-pi/2}"/>
       <geometry>
-        <mesh filename="package://htb_description/meshes/realsense.dae"/>
+        <mesh filename="file://$(find htb_description)/meshes/realsense.dae"/>
       </geometry>
       <material name="red"/>

Commit message: Update robot description

File: htb_description/urdf/htb.urdf.xacro (robot description, xacro)
@@ -1,151 +1,12 @@
-<?xml version="1.0" ?>
+<?xml version="1.0"?>
 <robot name="htb" xmlns:xacro="http://www.ros.org/wiki/xacro">
-  <xacro:include filename="$(find htb_description)/urdf/materials.urdf.xacro" />
-  <xacro:include filename="$(find htb_description)/urdf/mech/wheel.urdf.xacro" />
-  <xacro:include filename="$(find htb_description)/urdf/mech/caster.urdf.xacro" />
-  <xacro:property name="camera_link_size" value="0.05" /> <!-- Size of square 'camera' box -->
-  <xacro:arg name="use_ros2_control" default="false" />
-  <xacro:arg name="sim_mode" default="true" />
-  <link name="base_link">
-    <!-- pose and inertial -->
-    <pose>0 0 0.11 0 0 0</pose>
-    <inertia>
-      <mass value="2"/>
-      <origin rpy="0 0 0" xyz="0 0 0.11"/>
-      <inertia ixx="0.0395416666667" ixy="0" ixz="0" iyy="0.106208333333" iyz="0" izz="0.106208333333"/>
-    </inertia>
-    <!-- body -->
-    <collision name="collision_chassis">
-      <geometry>
-        <box size="0.53 0.38 0.02"/>
-      </geometry>
-    </collision>
-    <visual>
-      <origin rpy="0 0 0" xyz="0 0 0"/>
-      <geometry>
-        <box size="0.53 0.38 0.02"/>
-      </geometry>
-      <material name="blue"/>
-    </visual>
-  </link>
-  <!-- upper joint-->
-  <joint name="upper_joint" type="fixed">
-    <axis xyz="0 1 0" />
-    <origin xyz="0 0 0.14" rpy="0 0 0"/>
-    <parent link="base_link"/>
-    <child link="upper_link"/>
-  </joint>
-  <link name="upper_link">
-    <!-- pose and inertial -->
-    <pose>0
-      0 0.11 0 0 0</pose>
-    <inertial>
-      <mass value="2"/>
-      <origin rpy="0 0 0" xyz="0 0 0.11"/>
-      <inertia ixx="0.0395416666667" ixy="0" ixz="0" iyy="0.106208333333" iyz="0" izz="0.106208333333"/>
-    </inertial>
-    <!-- body -->
-    <visual>
-      <origin rpy="0 0 0" xyz="0 0 0"/>
-      <geometry>
-        <box size="0.53 0.38 0.02"/>
-      </geometry>
-      <material name="blue"/>
-    </visual>
-  </link>
-  <!-- RP-lidar joint-->
-  <joint name="rplidar_joint" type="fixed">
-    <axis xyz="0 1 0" />
-    <origin xyz="0.215 0 0.12" rpy="0 0 0"/>
-    <parent link="base_link"/>
-    <child link="rplidar_link"/>
-  </joint>
-  <!-- RP-lidar link-->
-  <link name="rplidar_link">
-    <collision>
-      <origin xyz="0 0 -0.06" rpy="0 0 ${pi}"/>
-      <geometry>
-        <mesh filename="file://$(find htb_description)/meshes/rplidar.dae"/>
-      </geometry>
-    </collision>
-    <visual>
-      <origin xyz="0 0 -0.06" rpy="0 0 ${pi}"/>
-      <geometry>
-        <mesh filename="file://$(find htb_description)/meshes/rplidar.dae"/>
-      </geometry>
-      <material name="red"/>
-    </visual>
-    <inertial>
-      <mass value="1e-5" />
-      <origin xyz="0 0 0" rpy="0 0 0"/>
-      <inertia ixx="1e-6" ixy="0" ixz="0" iyy="1e-6" iyz="0" izz="1e-6" />
-    </inertial>
-  </link>
-  <!-- Camera joint-->
-  <joint name="camera_joint" type="fixed">
-    <axis xyz="0 1 0" />
-    <origin xyz="0.22 0.08 0.10" rpy="0 0 0"/>
-    <parent link="base_link"/>
-    <child link="realsense_camera"/>
-  </joint>
-  <!-- Camera link-->
-  <link name="realsense_camera">
-    <collision>
-      <origin xyz="0.03 0 0" rpy="${-pi/2} 0 ${-pi/2}"/>
-      <geometry>
-        <mesh filename="file://$(find htb_description)/meshes/realsense.dae"/>
-      </geometry>
-    </collision>
-    <visual>
-      <origin xyz="0.03 0 0" rpy="${-pi/2} 0 ${-pi/2}"/>
-      <geometry>
-        <mesh filename="file://$(find htb_description)/meshes/realsense.dae"/>
-      </geometry>
-      <material name="red"/>
-    </visual>
-    <inertial>
-      <mass value="1e-5" />
-      <origin xyz="0 0 0" rpy="0 0 0"/>
-      <inertia ixx="1e-6" ixy="0" ixz="0" iyy="1e-6" iyz="0" izz="1e-6" />
-    </inertial>
-  </link>
-  <!-- generate an optical frame http://www.ros.org/reps/rep-0103.html#suffix-frames
-      so that ros and opencv can operate on the camera frame correctly -->
-  <joint name="camera_optical_joint" type="fixed">
-    <!-- these values have to be these values otherwise the gazebo camera image
-        won't be aligned properly with the frame it is supposedly originating from -->
-    <origin xyz="0 0 0" rpy="${-pi/2} 0 ${-pi/2}"/>
-    <parent link="realsense_camera"/>
-    <child link="realsense_link_optical"/>
-  </joint>
-  <link name="realsense_link_optical">
-  </link>
-  <joint name="realsense_mountpoint_joint" type="fixed">
-    <origin xyz="0 0 0" rpy="0 0 0"/>
-    <parent link="realsense_link_optical"/>
-    <child link="realsense_mount_point"/>
-  </joint>
-  <link name="realsense_mount_point">
-  </link>
-  <!-- -->
-  <!-- Right Wheel -->
-  <xacro:link_wheel name="right_wheel" />
-  <xacro:joint_wheel name="right_wheel_joint" child="right_wheel" origin_xyz="0.125 -0.2225 -0.04" />
-  <!-- Left Wheel -->
-  <xacro:link_wheel name="left_wheel" />
-  <xacro:joint_wheel name="left_wheel_joint" child="left_wheel" origin_xyz="0.125 0.2225 -0.04" />
-  <!-- Caster wheels -->
-  <xacro:caster_wheel name="left_caster" origin_xyz="-0.185 0.11 -0.06" wheel="l"/>
-  <xacro:caster_wheel name="right_caster" origin_xyz="-0.185 -0.11 -0.06" wheel="r"/>
-  <!-- Vertical supports -->
-  <xacro:vertical_support number="1" x="0.105"  y="0.17" />
-  <xacro:vertical_support number="2" x="0.105"  y="-0.17" />
-  <xacro:vertical_support number="3" x="-0.245" y="0.17"  />
-  <xacro:vertical_support number="4" x="-0.245" y="-0.17"  />
-  <xacro:if value="$(arg use_ros2_control)">
-    <xacro:include filename="$(find htb_description)/urdf/ros2_control.xacro" />
-  </xacro:if>
-  <xacro:unless value="$(arg use_ros2_control)">
-    <xacro:include filename="$(find htb_description)/urdf/gazebo_control.xacro" />
-  </xacro:unless>
+  <!-- Import htb description -->
+  <xacro:include filename="$(find htb_description)/urdf/htb_description.urdf.xacro" />
+  <!-- Import Rviz colors -->
+  <xacro:include filename="$(find htb_description)/gazebo/htb.materials.xacro" />
+  <!-- Import diffbot ros2_control description -->
+  <xacro:include filename="$(find htb_description)/ros2_control/htb.ros2_control.xacro" />
+  <!-- class instantiation -->
+  <xacro:htb_robot />
+  <xacro:htb_ros2_control />
 </robot>

File: htb_description/urdf/mech/wheel.urdf.xacro (robot description, xacro)
@@ -28,4 +28,5 @@
         <parent link="base_link"/>
         <axis rpy="0 0 0" xyz="0 1 0"/>
+        <dynamics damping="0.2"/>
       </joint>
     </xacro:macro>
