Commit message: Add base_footprint

File: htb_description/urdf/htb.urdf (robot description, URDF)
Before this commit: robot htb, 18 links, 17 joints
Links:
- added link base_footprint
- link caster_l_hubcap: geometry visual mesh filename=file:///home/aresuser/ros2_ws/install/htb_description/share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
- link caster_l_swivel: geometry visual mesh filename=file:///home/aresuser/ros2_ws/install/htb_description/share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
- link caster_l_wheel: geometry collision mesh filename=file:///home/aresuser/ros2_ws/install/htb_description/share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; visual mesh filename=file:///home/aresuser/ros2_ws/install/htb_description/share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
- link caster_r_hubcap: geometry visual mesh filename=file:///home/aresuser/ros2_ws/install/htb_description/share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
- link caster_r_swivel: geometry visual mesh filename=file:///home/aresuser/ros2_ws/install/htb_description/share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
- link caster_r_wheel: geometry collision mesh filename=file:///home/aresuser/ros2_ws/install/htb_description/share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; visual mesh filename=file:///home/aresuser/ros2_ws/install/htb_description/share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
- link realsense_camera: geometry collision mesh filename=file:///home/aresuser/ros2_ws/install/htb_description/share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; visual mesh filename=file:///home/aresuser/ros2_ws/install/htb_description/share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
- link rplidar_link: geometry collision mesh filename=file:///home/aresuser/ros2_ws/install/htb_description/share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; visual mesh filename=file:///home/aresuser/ros2_ws/install/htb_description/share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
Joints:
- added joint base_footprint_joint: type fixed, parent base_link, child base_footprint, origin xyz=0 0 -0.11 rpy=0 0 0, axis 0 1 0

File: htb_description/urdf/htb_description.urdf.xacro (robot description, xacro)
@@ -29,4 +29,21 @@
       </visual>
     </link>
+    <link name="base_footprint">
+      <!-- pose and inertial -->
+      <pose>0 0 0 0 0 0</pose>
+      <inertia>
+        <mass value="0.01" />
+        <origin rpy="0 0 0" xyz="0 0 0.11" />
+        <inertia ixx="0.0395416666667" ixy="0" ixz="0" iyy="0.106208333333" iyz="0"
+          izz="0.106208333333" />
+      </inertia>
+    </link>
+    <!-- base_footrpint joint-->
+    <joint name="base_footprint_joint" type="fixed">
+      <axis xyz="0 1 0" />
+      <origin xyz="0 0 -0.11" rpy="0 0 0" />
+      <parent link="base_link" />
+      <child link="base_footprint" />
+    </joint>
     <!-- upper joint-->
     <joint name="upper_joint" type="fixed">
