Commit message: Update robot description

File: htb_description/install/htb_description/share/htb_description/urdf/htb.urdf.xacro (robot description, xacro)
@@ -9,9 +9,9 @@
     <!-- pose and inertial -->
     <pose>0 0 0.11 0 0 0</pose>
-    <inertia>
+    <inertial>
       <mass value="2"/>
       <origin rpy="0 0 0" xyz="0 0 0.11"/>
       <inertia ixx="0.0395416666667" ixy="0" ixz="0" iyy="0.106208333333" iyz="0" izz="0.106208333333"/>
-    </inertia>
+    </inertial>
     <!-- body -->
     <collision name="collision_chassis">
