Commit message: Update robot description

File: htb_description/gazebo/htb.gazebo.xacro (robot description, xacro)
@@ -3,5 +3,5 @@
   <xacro:macro name="htb_gazebo">
     <!-- camera -->
-    <gazebo reference="realsense_link_optical">
+    <gazebo>
       <plugin name="diff_drive" filename="libgazebo_ros_diff_drive.so">
         <!-- Wheel Information -->

File: htb_description/urdf/htb_description.urdf.xacro (robot description, xacro)
@@ -137,4 +137,7 @@
       <material>Gazebo/Orange</material>
     </gazebo>
+    <gazebo reference="upper_link">
+      <material>Gazebo/Orange</material>
+    </gazebo>
     <!-- Right Wheel -->
     <xacro:link_wheel name="right_wheel" />

File: htb_description/urdf/htb_gazebo.urdf.xacro (robot description, xacro)
@@ -15,4 +15,4 @@
   <!-- class instantiation -->
   <xacro:htb_robot />
-  <!-- <xacro:htb_gazebo /> -->
+  <xacro:htb_gazebo />
 </robot>

File: htb_description/urdf/mech/caster.urdf.xacro (robot description, xacro)
@@ -3,74 +3,83 @@
   <xacro:macro name="caster_wheel" params="name origin_xyz wheel">
     <!-- Caster -->
+    <gazebo reference="caster_${wheel}_swivel">
+      <material>Gazebo/Black</material>
+    </gazebo>
     <joint name="base_caster_${wheel}_swivel_joint" type="continuous">
-      <origin rpy=" 0 0 0" xyz="${origin_xyz}"/>
-      <anchor xyz="0 0 0"/>
+      <origin rpy=" 0 0 0" xyz="${origin_xyz}" />
+      <anchor xyz="0 0 0" />
       <limit effort="100" velocity="100" k_velocity="0" />
       <joint_properties damping="0.0" friction="0.0" />
-      <parent link="base_link"/>
-        <axis rpy="0 0 0" xyz="0 0 1"/>
-      <child link="caster_${wheel}_swivel"/>
+      <parent link="base_link" />
+      <axis rpy="0 0 0" xyz="0 0 1" />
+      <child link="caster_${wheel}_swivel" />
     </joint>
     <link name="caster_${wheel}_swivel">
       <inertial>
-        <mass value="0.1"/>
-        <origin xyz="0 0 0"/>
+        <mass value="0.1" />
+        <origin xyz="0 0 0" />
         <inertia ixx="0.01" ixy="0" ixz="0"
-          iyy="0.01" iyz="0" izz="0.01"/>
+          iyy="0.01" iyz="0" izz="0.01" />
       </inertial>
       <visual>
-        <origin xyz="0 0 0" rpy="0 0 0"/>
+        <origin xyz="0 0 0" rpy="0 0 0" />
         <geometry name="base_link">
           <mesh filename="file://$(find htb_description)/meshes/caster_swivel.stl" />
         </geometry>
-        <material name="blue"/>
+        <material name="blue" />
       </visual>
     </link>
+    <gazebo reference="caster_${wheel}_hubcap">
+      <material>Gazebo/Grey</material>
+    </gazebo>
     <!-- Center Wheel + Hubcap -->
     <link name="caster_${wheel}_hubcap">
       <inertial>
-        <mass value="0.01"/>
-        <origin xyz="0 0 0"/>
+        <mass value="0.01" />
+        <origin xyz="0 0 0" />
         <inertia ixx="0.012411765597" ixy="-0.000711733678" ixz="0.00050272983"
-          iyy="0.015218160428" iyz="-0.000004273467" izz="0.011763977943"/>
+          iyy="0.015218160428" iyz="-0.000004273467" izz="0.011763977943" />
       </inertial>
       <visual>
-        <origin xyz="0 0 0" rpy="0 0 0"/>
+        <origin xyz="0 0 0" rpy="0 0 0" />
         <geometry name="base_link">
           <mesh filename="file://$(find htb_description)/meshes/caster_hubcap.stl" />
         </geometry>
-        <material name="blue"/>
+        <material name="blue" />
       </visual>
     </link>
     <joint name="caster_${wheel}_swivel_hubcap_joint" type="continuous">
-      <origin xyz="-0.026 0 -0.016" rpy="0 0 0"/>
-      <axis xyz="0 1 0"/>
-      <anchor xyz="0 0 0"/>
+      <origin xyz="-0.026 0 -0.016" rpy="0 0 0" />
+      <axis xyz="0 1 0" />
+      <anchor xyz="0 0 0" />
       <limit effort="100" velocity="100" k_velocity="0" />
       <joint_properties damping="0.0" friction="0.0" />
-      <parent link="caster_${wheel}_swivel"/>
-      <child link="caster_${wheel}_wheel"/>
+      <parent link="caster_${wheel}_swivel" />
+      <child link="caster_${wheel}_wheel" />
     </joint>
+    <gazebo reference="caster_${wheel}_wheel">
+      <material>Gazebo/Black</material>
+    </gazebo>
     <link name="caster_${wheel}_wheel">
       <inertial>
-        <mass value="0.1"/>
-        <origin xyz="0 0 0"/>
+        <mass value="0.1" />
+        <origin xyz="0 0 0" />
         <inertia ixx="0.012411765597" ixy="-0.000711733678" ixz="0.00050272983"
-          iyy="0.015218160428" iyz="-0.000004273467" izz="0.011763977943"/>
+          iyy="0.015218160428" iyz="-0.000004273467" izz="0.011763977943" />
       </inertial>
       <visual>
-        <origin xyz="0 0 0" rpy="0 0 0"/>
+        <origin xyz="0 0 0" rpy="0 0 0" />
         <geometry name="base_link">
           <mesh filename="file://$(find htb_description)/meshes/caster_wheel.stl" />
         </geometry>
         <material name="WheelBlack">
-          <color rgba="0.117 0.117 0.117 1"/>
+          <color rgba="0.117 0.117 0.117 1" />
         </material>
       </visual>
       <collision>
-        <origin xyz="0 0 0" rpy="0 0 0"/>
+        <origin xyz="0 0 0" rpy="0 0 0" />
         <geometry>
           <mesh filename="file://$(find htb_description)/meshes/caster_wheel.stl" />
-          <cylinder radius="0.0375" length="0.01"/>
+          <cylinder radius="0.0375" length="0.01" />
         </geometry>
         <surface>
@@ -87,7 +96,7 @@
     </link>
     <joint name="caster_${wheel}_wheel_joint" type="fixed">
-      <origin xyz="-0.0035 0 -0.001" rpy="0 0 0"/>
-      <parent link="caster_${wheel}_wheel"/>
-      <child link="caster_${wheel}_hubcap"/>
+      <origin xyz="-0.0035 0 -0.001" rpy="0 0 0" />
+      <parent link="caster_${wheel}_wheel" />
+      <child link="caster_${wheel}_hubcap" />
     </joint>
   </xacro:macro>

File: htb_description/urdf/mech/wheel.urdf.xacro (robot description, xacro)
@@ -1,65 +1,71 @@
 <?xml version="1.0"?>
 <robot xmlns:xacro="http://www.ros.org/wiki/xacro">
-    <xacro:macro name="link_wheel" params="name">
-        <link name="${name}">
-            <inertial>
-              <mass value="0.5"/>
-              <origin rpy="0 1.5707 1.5707" xyz="0 0 0"/>
-              <inertia ixx="0.000526666666667" ixy="0" ixz="0" iyy="0.000526666666667" iyz="0" izz="0.001"/>
-            </inertial>
-            <collision name="link_${name}_collision">
-              <origin rpy="0 1.5707 1.5707" xyz="0 0 0"/>
-              <geometry>
-                <cylinder length="0.045" radius="0.08"/>
-              </geometry>
-            </collision>
-            <visual name="${name}_visual">
-              <origin rpy="0 1.5707 1.5707" xyz="0 0 0"/>
-              <geometry>
-                <cylinder length="0.045" radius="0.08"/>
-              </geometry>
-            </visual>
-        </link>
-    </xacro:macro>
-    <xacro:macro name="joint_wheel" params="name child origin_xyz">
-      <joint name="${name}" type="continuous">
-        <origin rpy="0 0 0" xyz="${origin_xyz}"/>
-        <child link="${child}"/>
-        <parent link="base_link"/>
-        <axis rpy="0 0 0" xyz="0 1 0"/>
-        <dynamics damping="0.2"/>
-      </joint>
-    </xacro:macro>
-    <xacro:macro name="cylinder_inertia" params="mass r l">
-      <inertia  ixx="${mass*(3*r*r+l*l)/12}" ixy = "0" ixz = "0"
-                iyy="${mass*(3*r*r+l*l)/12}" iyz = "0"
-                izz="${mass*(r*r)/2}" />
-    </xacro:macro>
-    <xacro:macro name="vertical_support" params="number x y">
-      <link name="support_${number}">
-        <inertial>
-          <mass value="0.1"/>
-          <origin xyz="0 0 0" rpy="0 0 0"/>
-          <inertia ixx="0.000526666666667" ixy="0" ixz="0" iyy="0.000526666666667" iyz="0" izz="0.001"/>
-        </inertial>
-        <collision name="vertical_support_${number}_collision">
-          <origin xyz="0 0 0" rpy="0 0 0"/>
-          <geometry>
-            <box size="0.04 0.04 0.12"/>
-          </geometry>
-        </collision>
-        <visual name="support_${number}_visual">
-          <origin xyz="0 0 0" rpy="0 0 0"/>
-          <geometry>
-            <box size="0.04 0.04 0.12"/>
-          </geometry>
-        </visual>
-      </link>
-      <joint name="support_${number}_joint" type="fixed">
-        <axis xyz="0 0 1" />
-        <origin rpy="0 0 0" xyz="${x} ${y} 0.07"/>
-        <parent link="base_link"/>
-        <child link="support_${number}"/>
-      </joint>
-    </xacro:macro>
-  </robot>
+  <xacro:macro name="link_wheel" params="name">
+    <gazebo reference="${name}">
+      <material>Gazebo/Grey</material>
+    </gazebo>
+    <link name="${name}">
+      <inertial>
+        <mass value="0.5" />
+        <origin rpy="0 1.5707 1.5707" xyz="0 0 0" />
+        <inertia ixx="0.000526666666667" ixy="0" ixz="0" iyy="0.000526666666667" iyz="0" izz="0.001" />
+      </inertial>
+      <collision name="link_${name}_collision">
+        <origin rpy="0 1.5707 1.5707" xyz="0 0 0" />
+        <geometry>
+          <cylinder length="0.045" radius="0.08" />
+        </geometry>
+      </collision>
+      <visual name="${name}_visual">
+        <origin rpy="0 1.5707 1.5707" xyz="0 0 0" />
+        <geometry>
+          <cylinder length="0.045" radius="0.08" />
+        </geometry>
+      </visual>
+    </link>
+  </xacro:macro>
+  <xacro:macro name="joint_wheel" params="name child origin_xyz">
+    <joint name="${name}" type="continuous">
+      <origin rpy="0 0 0" xyz="${origin_xyz}" />
+      <child link="${child}" />
+      <parent link="base_link" />
+      <axis rpy="0 0 0" xyz="0 1 0" />
+      <dynamics damping="0.2" />
+    </joint>
+  </xacro:macro>
+  <xacro:macro name="cylinder_inertia" params="mass r l">
+    <inertia ixx="${mass*(3*r*r+l*l)/12}" ixy="0" ixz="0"
+      iyy="${mass*(3*r*r+l*l)/12}" iyz="0"
+      izz="${mass*(r*r)/2}" />
+  </xacro:macro>
+  <xacro:macro name="vertical_support" params="number x y">
+    <gazebo reference="support_${number}">
+      <material>Gazebo/Black</material>
+    </gazebo>
+    <link name="support_${number}">
+      <inertial>
+        <mass value="0.1" />
+        <origin xyz="0 0 0" rpy="0 0 0" />
+        <inertia ixx="0.000526666666667" ixy="0" ixz="0" iyy="0.000526666666667" iyz="0" izz="0.001" />
+      </inertial>
+      <collision name="vertical_support_${number}_collision">
+        <origin xyz="0 0 0" rpy="0 0 0" />
+        <geometry>
+          <box size="0.04 0.04 0.12" />
+        </geometry>
+      </collision>
+      <visual name="support_${number}_visual">
+        <origin xyz="0 0 0" rpy="0 0 0" />
+        <geometry>
+          <box size="0.04 0.04 0.12" />
+        </geometry>
+      </visual>
+    </link>
+    <joint name="support_${number}_joint" type="fixed">
+      <axis xyz="0 0 1" />
+      <origin rpy="0 0 0" xyz="${x} ${y} 0.07" />
+      <parent link="base_link" />
+      <child link="support_${number}" />
+    </joint>
+  </xacro:macro>
+</robot>
