Commit message: Update robot description

File: htb_description/ros2_control/htb.ros2_control.xacro (robot description, xacro)
@@ -5,5 +5,5 @@
     <ros2_control name="GazeboSystem" type="system">
       <hardware>
-        <plugin>gazebo_ros2_control/GazeboSystem</plugin>
+        <plugin>htb_hardware_interfaces/HtbSystem</plugin>
       </hardware>
       <joint name="left_wheel_joint">

File: htb_description/urdf/htb_description.urdf.xacro (robot description, xacro)
@@ -139,22 +139,15 @@
     <!-- Right Wheel -->
     <xacro:link_wheel name="right_wheel" />
-    <xacro:joint_wheel
-      name="right_wheel_joint" child="right_wheel" origin_xyz="0.125 -0.2225 -0.04" /> --> <!-- Left
-    Wheel -->
-    <xacro:link_wheel
-      name="left_wheel" />
-    <xacro:joint_wheel name="left_wheel_joint" child="left_wheel"
-      origin_xyz="0.125 0.2225 -0.04" />
+    <xacro:joint_wheel name="right_wheel_joint" child="right_wheel" origin_xyz="0.125 -0.2225 -0.04" />
+    <!-- Left Wheel -->
+    <xacro:link_wheel name="left_wheel" />
+    <xacro:joint_wheel name="left_wheel_joint" child="left_wheel" origin_xyz="0.125 0.2225 -0.04" />
     <!-- Caster wheels -->
-    <xacro:caster_wheel name="left_caster"
-      origin_xyz="-0.185 0.11 -0.06" wheel="l" />
-    <xacro:caster_wheel name="right_caster"
-      origin_xyz="-0.185 -0.11 -0.06" wheel="r" />
+    <xacro:caster_wheel name="left_caster" origin_xyz="-0.185 0.11 -0.06" wheel="l" />
+    <xacro:caster_wheel name="right_caster" origin_xyz="-0.185 -0.11 -0.06" wheel="r" />
     <!-- Vertical supports -->
-    <xacro:vertical_support number="1" x="0.105"
-      y="0.17" />
+    <xacro:vertical_support number="1" x="0.105" y="0.17" />
     <xacro:vertical_support number="2" x="0.105" y="-0.17" />
-    <xacro:vertical_support
-      number="3" x="-0.245" y="0.17" />
+    <xacro:vertical_support number="3" x="-0.245" y="0.17" />
     <xacro:vertical_support number="4" x="-0.245" y="-0.17" />
   </xacro:macro>

File: htb_description/urdf/mech/wheel.urdf.xacro (robot description, xacro)
@@ -8,5 +8,5 @@
               <inertia ixx="0.000526666666667" ixy="0" ixz="0" iyy="0.000526666666667" iyz="0" izz="0.001"/>
             </inertial>
-            <collision name="link_right_wheel_collision">
+            <collision name="link_${name}_collision">
               <origin rpy="0 1.5707 1.5707" xyz="0 0 0"/>
               <geometry>

Commit message: Update robot description

File: htb_description/ros2_control/htb.ros2_control.xacro (robot description, xacro)
@@ -12,6 +12,6 @@
           <param name="max">10</param>
         </command_interface>
+        <state_interface name="position" />
         <state_interface name="velocity" />
-        <state_interface name="position" />
       </joint>
       <joint name="right_wheel_joint">
@@ -20,6 +20,6 @@
           <param name="max">10</param>
         </command_interface>
+        <state_interface name="position" />
         <state_interface name="velocity" />
-        <state_interface name="position" />
       </joint>
     </ros2_control>

File: htb_description/urdf/htb_description.urdf.xacro (robot description, xacro)
@@ -145,5 +145,5 @@
     <!-- Caster wheels -->
     <xacro:caster_wheel name="left_caster" origin_xyz="-0.185 0.11 -0.06" wheel="l" />
-    <xacro:caster_wheel name="right_caster" origin_xyz="-0.185 -0.11 -0.06" wheel="r" />
+    <!-- <xacro:caster_wheel name="right_caster" origin_xyz="-0.185 -0.11 -0.06" wheel="r" /> -->
     <!-- Vertical supports -->
     <xacro:vertical_support number="1" x="0.105" y="0.17" />

File: htb_description/urdf/mech/caster_fixed.urdf.xacro (robot description, xacro)
@@ -22,5 +22,5 @@
         <origin xyz="0 0 0" rpy="0 0 0"/>
         <geometry name="base_link">
-          <mesh filename="file://$(find htb_description)/meshes/caster_swivel.stl" />
+          <mesh filename="package://htb_description/meshes/caster_swivel.stl"/>
         </geometry>
         <material name="blue"/>
@@ -38,5 +38,5 @@
         <origin xyz="0 0 0" rpy="0 0 0"/>
         <geometry name="base_link">
-          <mesh filename="file://$(find htb_description)/meshes/caster_hubcap.stl" />
+          <mesh filename="package://htb_description/meshes/caster_hubcap.stl"/>
         </geometry>
         <material name="blue"/>
@@ -62,5 +62,5 @@
         <origin xyz="0 0 0" rpy="0 0 0"/>
         <geometry name="base_link">
-          <mesh filename="file://$(find htb_description)/meshes/caster_wheel.stl" />
+          <mesh filename="package://htb_description/meshes/caster_wheel.stl"/>
         </geometry>
         <material name="WheelBlack">
@@ -69,7 +69,8 @@
       </visual>
       <collision>
+        <!-- <origin xyz="0 0 0" rpy="${-3.1415927/2.0} 0 0"/> -->
         <origin xyz="0 0 0" rpy="0 0 0"/>
         <geometry>
-          <mesh filename="file://$(find htb_description)/meshes/caster_wheel.stl" />
+          <mesh filename="package://htb_description/meshes/caster_wheel.stl"/>
           <cylinder radius="0.0375" length="0.01"/>
         </geometry>

Commit message: Update robot description

File: htb_description/ros2_control/htb.ros2_control.xacro (robot description, xacro)
@@ -5,5 +5,5 @@
     <ros2_control name="GazeboSystem" type="system">
       <hardware>
-        <plugin>mock_components/GenericSystem</plugin>
+        <plugin>htb_hardware/HtbSystemHardware</plugin>
       </hardware>
       <joint name="left_wheel_joint">

File: htb_description/urdf/htb.urdf.xacro (robot description, xacro)
@@ -1,4 +1,5 @@
 <?xml version="1.0"?>
 <robot name="htb" xmlns:xacro="http://www.ros.org/wiki/xacro">
+  <xacro:arg name="fixed_caster" default="false" />
   <!-- Import htb description -->
   <xacro:include filename="$(find htb_description)/urdf/htb_description.urdf.xacro" />
@@ -8,5 +9,5 @@
   <xacro:include filename="$(find htb_description)/ros2_control/htb.ros2_control.xacro" />
   <!-- class instantiation -->
-  <xacro:htb_robot />
+  <xacro:htb_robot fixed_caster="$(arg fixed_caster)"/>
   <xacro:htb_ros2_control />
 </robot>

File: htb_description/urdf/htb_description.urdf.xacro (robot description, xacro)
@@ -1,7 +1,8 @@
 <?xml version="1.0"?>
 <robot xmlns:xacro="http://www.ros.org/wiki/xacro">
-  <xacro:macro name="htb_robot">
+  <xacro:macro name="htb_robot" params="fixed_caster">
     <xacro:include filename="$(find htb_description)/urdf/mech/wheel.urdf.xacro" />
     <xacro:include filename="$(find htb_description)/urdf/mech/caster.urdf.xacro" />
+    <xacro:include filename="$(find htb_description)/urdf/mech/caster_fixed.urdf.xacro" />
     <xacro:property name="camera_link_size" value="0.05" /> <!-- Size of square 'camera' box -->
     <link name="base_link">
@@ -147,6 +148,12 @@
     <xacro:joint_wheel name="left_wheel_joint" child="left_wheel" origin_xyz="0.125 0.2225 -0.04" />
     <!-- Caster wheels -->
-    <xacro:caster_wheel name="left_caster" origin_xyz="-0.185 0.11 -0.06" wheel="l" />
-    <xacro:caster_wheel name="right_caster" origin_xyz="-0.185 -0.11 -0.06" wheel="r" />
+    <xacro:if value="$(arg fixed_caster)">
+      <xacro:caster_wheel_fixed name="left_caster" origin_xyz="-0.185 0.11 -0.06" wheel="l" />
+      <xacro:caster_wheel_fixed name="right_caster" origin_xyz="-0.185 -0.11 -0.06" wheel="r" />
+    </xacro:if>
+    <xacro:unless value="$(arg fixed_caster)">
+      <xacro:caster_wheel name="left_caster" origin_xyz="-0.185 0.11 -0.06" wheel="l" />
+      <xacro:caster_wheel name="right_caster" origin_xyz="-0.185 -0.11 -0.06" wheel="r" />
+    </xacro:unless>
     <!-- Vertical supports -->
     <xacro:vertical_support number="1" x="0.105" y="0.17" />

File: htb_description/urdf/htb_gazebo.urdf.xacro (robot description, xacro)
@@ -6,5 +6,5 @@
 -->
 <robot xmlns:xacro="http://www.ros.org/wiki/xacro" name="htb_robot">
-  <xacro:arg name="use_gazebo" default="false" />
+  <xacro:arg name="fixed_caster" default="false" />
   <!-- Import htb description -->
   <xacro:include filename="$(find htb_description)/urdf/htb_description.urdf.xacro" />
@@ -14,5 +14,5 @@
   <xacro:include filename="$(find htb_description)/gazebo/htb.materials.xacro" />
   <!-- class instantiation -->
-  <xacro:htb_robot />
+  <xacro:htb_robot fixed_caster="$(arg fixed_caster)"/>
   <xacro:htb_gazebo />
 </robot>

File: htb_description/urdf/mech/caster_fixed.urdf.xacro (robot description, xacro)
@@ -1,77 +1,85 @@
 <?xml version="1.0"?>
 <robot xmlns:xacro="http://www.ros.org/wiki/xacro">
-  <xacro:macro name="caster_wheel" params="name origin_xyz wheel">
+  <xacro:macro name="caster_wheel_fixed" params="name origin_xyz wheel">
     <!-- Caster -->
-    <joint name="base_caster_${wheel}_swivel_joint" type="continuous">
-      <origin rpy=" 0 0 0" xyz="${origin_xyz}"/>
-      <anchor xyz="0 0 0"/>
+    <gazebo reference="caster_${wheel}_swivel">
+      <material>Gazebo/Black</material>
+    </gazebo>
+    <joint name="base_caster_${wheel}_swivel_joint" type="fixed">
+      <origin rpy=" 0 0 0" xyz="${origin_xyz}" />
+      <anchor xyz="0 0 0" />
       <limit effort="100" velocity="100" k_velocity="0" />
       <joint_properties damping="0.0" friction="0.0" />
-      <parent link="base_link"/>
-        <axis rpy="0 0 0" xyz="0 0 1"/>
-      <child link="caster_${wheel}_swivel"/>
+      <parent link="base_link" />
+      <axis rpy="0 0 0" xyz="0 0 1" />
+      <child link="caster_${wheel}_swivel" />
     </joint>
     <link name="caster_${wheel}_swivel">
       <inertial>
-        <mass value="0.1"/>
-        <origin xyz="0 0 0"/>
+        <mass value="0.1" />
+        <origin xyz="0 0 0" />
         <inertia ixx="0.01" ixy="0" ixz="0"
-          iyy="0.01" iyz="0" izz="0.01"/>
+          iyy="0.01" iyz="0" izz="0.01" />
       </inertial>
       <visual>
-        <origin xyz="0 0 0" rpy="0 0 0"/>
+        <origin xyz="0 0 0" rpy="0 0 0" />
         <geometry name="base_link">
-          <mesh filename="package://htb_description/meshes/caster_swivel.stl"/>
+          <mesh filename="file://$(find htb_description)/meshes/caster_swivel.stl" />
         </geometry>
-        <material name="blue"/>
+        <material name="blue" />
       </visual>
     </link>
+    <gazebo reference="caster_${wheel}_hubcap">
+      <material>Gazebo/Grey</material>
+    </gazebo>
     <!-- Center Wheel + Hubcap -->
     <link name="caster_${wheel}_hubcap">
       <inertial>
-        <mass value="0.01"/>
-        <origin xyz="0 0 0"/>
+        <mass value="0.01" />
+        <origin xyz="0 0 0" />
         <inertia ixx="0.012411765597" ixy="-0.000711733678" ixz="0.00050272983"
-          iyy="0.015218160428" iyz="-0.000004273467" izz="0.011763977943"/>
+          iyy="0.015218160428" iyz="-0.000004273467" izz="0.011763977943" />
       </inertial>
       <visual>
-        <origin xyz="0 0 0" rpy="0 0 0"/>
+        <origin xyz="0 0 0" rpy="0 0 0" />
         <geometry name="base_link">
-          <mesh filename="package://htb_description/meshes/caster_hubcap.stl"/>
+          <mesh filename="file://$(find htb_description)/meshes/caster_hubcap.stl" />
         </geometry>
-        <material name="blue"/>
+        <material name="blue" />
       </visual>
     </link>
-    <joint name="caster_${wheel}_swivel_hubcap_joint" type="continuous">
-      <origin xyz="-0.026 0 -0.016" rpy="0 0 0"/>
-      <axis xyz="0 1 0"/>
-      <anchor xyz="0 0 0"/>
+    <joint name="caster_${wheel}_swivel_hubcap_joint" type="fixed">
+      <origin xyz="-0.026 0 -0.016" rpy="0 0 0" />
+      <axis xyz="0 1 0" />
+      <anchor xyz="0 0 0" />
       <limit effort="100" velocity="100" k_velocity="0" />
       <joint_properties damping="0.0" friction="0.0" />
-      <parent link="caster_${wheel}_swivel"/>
-      <child link="caster_${wheel}_wheel"/>
+      <parent link="caster_${wheel}_swivel" />
+      <child link="caster_${wheel}_wheel" />
     </joint>
+    <gazebo reference="caster_${wheel}_wheel">
+      <material>Gazebo/Black</material>
+    </gazebo>
     <link name="caster_${wheel}_wheel">
       <inertial>
-        <mass value="0.1"/>
-        <origin xyz="0 0 0"/>
+        <mass value="0.1" />
+        <origin xyz="0 0 0" />
         <inertia ixx="0.012411765597" ixy="-0.000711733678" ixz="0.00050272983"
-          iyy="0.015218160428" iyz="-0.000004273467" izz="0.011763977943"/>
+          iyy="0.015218160428" iyz="-0.000004273467" izz="0.011763977943" />
       </inertial>
       <visual>
-        <origin xyz="0 0 0" rpy="0 0 0"/>
+        <origin xyz="0 0 0" rpy="0 0 0" />
         <geometry name="base_link">
-          <mesh filename="package://htb_description/meshes/caster_wheel.stl"/>
+          <mesh filename="file://$(find htb_description)/meshes/caster_wheel.stl" />
         </geometry>
         <material name="WheelBlack">
-          <color rgba="0.117 0.117 0.117 1"/>
+          <color rgba="0.117 0.117 0.117 1" />
         </material>
       </visual>
       <collision>
-        <!-- <origin xyz="0 0 0" rpy="${-3.1415927/2.0} 0 0"/> -->
-        <origin xyz="0 0 0" rpy="0 0 0"/>
+        <origin xyz="0 0 0" rpy="0 0 0" />
         <geometry>
-          <mesh filename="package://htb_description/meshes/caster_wheel.stl"/>
-          <cylinder radius="0.0375" length="0.01"/>
+          <mesh filename="file://$(find htb_description)/meshes/caster_wheel.stl" />
+          <cylinder radius="0.0375" length="0.01" />
         </geometry>
         <surface>
@@ -88,7 +96,7 @@
     </link>
     <joint name="caster_${wheel}_wheel_joint" type="fixed">
-      <origin xyz="-0.0035 0 -0.001" rpy="0 0 0"/>
-      <parent link="caster_${wheel}_wheel"/>
-      <child link="caster_${wheel}_hubcap"/>
+      <origin xyz="-0.0035 0 -0.001" rpy="0 0 0" />
+      <parent link="caster_${wheel}_wheel" />
+      <child link="caster_${wheel}_hubcap" />
     </joint>
   </xacro:macro>
